File: 2x2/Handdrawnv1.kicad_pcb (KiCad board)
At the start: 2 copper layers, 63 x 42 mm, 24 parts, among them J2 USB_B_Mini, K1 KEYSW, K2 KEYSW, K3 KEYSW, K4 KEYSW, SW1 SW_PUSH, U1 ATMEGA32U4, Y2 Crystal_GND24_Small

Commit message: almost finished the 2x2, will be working on the 65 now
Parts:
- added F1: 500mA, Fuse:Fuse_1206_3216Metric_Pad1.42x1.75mm_HandSolder, B.Cu at (143.7, 58.6)
- C8: value 4.7uF -> 10uf
- SW1: footprint Button_Switch_SMD:SW_SPST_TL3342 -> Button_Switch_SMD:SW_SPST_SKQG_WithStem
- moved J2 4.69 mm to (148.8, 52.2)
- moved C6 2.90 mm to (141.6, 80.6)
- moved SW1 1.22 mm to (159.7, 61.1)
- moved C3 1.20 mm to (151.9, 65.8)
- moved R1 1.20 mm to (157.4, 66.2)
- moved R3 0.51 mm to (147.3, 63.0)
- moved R4 0.41 mm to (149.2, 63.0)
Connections:
- net Net-(J2-D+) renamed /USBD2+
- net Net-(J2-D-) renamed /USBD2-
- net Net-(U1-D+) renamed /USBD+
- net Net-(U1-D-) renamed /USBD-
- net Net-(U1-UCap) renamed /Ucap
- net Net-(U1-XTAL1) renamed /Xtal1
- net Net-(U1-XTAL2) renamed /Xtal2
- net Net-(U1-~{HWB/PE2}) renamed /HWB
- net Net-(U1-~{RESET}) renamed /Reset
- C4 pad 1: VCC -> +5V
- C5 pad 1: VCC -> +5V
- C6 pad 1: VCC -> +5V
- C7 pad 1: VCC -> +5V
- C8 pad 1: VCC -> +5V
- J2 pad 6: GND -> Earth
- R1 pad 1: VCC -> +5V
- U1 pad 14: VCC -> +5V
- U1 pad 2: VCC -> +5V
- U1 pad 24: VCC -> +5V
- U1 pad 34: VCC -> +5V
- U1 pad 44: VCC -> +5V
- U1 pad 7: VCC -> +5V
Routing:
- net +5V: track 0.00 -> 115.4 mm, vias 0 -> 6
- net VCC: track 111.0 -> 5.20 mm, vias 4 -> 0
- net GND: track 38.7 -> 30.7 mm, vias 22 -> 18
- net /USBD2-: track 2.84 -> 7.88 mm
- net /USBD2+: track 2.93 -> 7.88 mm
- net /Ucap: track 3.20 -> 4.25 mm
- net /Reset: track 18.5 -> 19.4 mm
- added copper zone on B.Cu, net Earth
- added copper zone on F.Cu, net Earth
Other:
- board size 63 x 42 mm -> 63 x 46.3 mm
