File: 65/65.kicad_sch (KiCad schematic)
At the start: 133 parts, among them K1 KEYSW, K10 KEYSW, K11 KEYSW, K12 KEYSW, K13 KEYSW, K14 KEYSW, K15 KEYSW, K16 KEYSW, K17 KEYSW, K18 KEYSW, K19 KEYSW, K2 KEYSW, K20 KEYSW, K21 KEYSW, K22 KEYSW, K23 KEYSW, K24 KEYSW, K25 KEYSW, K26 KEYSW, K27 KEYSW, K28 KEYSW, K29 KEYSW, K3 KEYSW, K30 KEYSW, K31 KEYSW, K32 KEYSW, K33 KEYSW, K34 KEYSW, K35 KEYSW, K36 KEYSW, K37 KEYSW, K38 KEYSW, K39 KEYSW, K4 KEYSW, K40 KEYSW, K41 KEYSW, K42 KEYSW, K43 KEYSW, K44 KEYSW, K45 KEYSW, K46 KEYSW, K47 KEYSW, K48 KEYSW, K49 KEYSW, K5 KEYSW, K50 KEYSW, K51 KEYSW, K52 KEYSW, K53 KEYSW, K54 KEYSW, K55 KEYSW, K56 KEYSW, K57 KEYSW, K58 KEYSW, K59 KEYSW, K6 KEYSW, K60 KEYSW, K61 KEYSW, K62 KEYSW, K63 KEYSW, K64 KEYSW, K65 KEYSW, K66 KEYSW, K7 KEYSW, K8 KEYSW, K9 KEYSW, U2 ATmega32U4-A

Commit message: almost finished the 2x2, will be working on the 65 now
Parts:
- added C1, C2, C3: 0.1uf, Capacitor_SMD:C_0805_2012Metric, symbol Device:C
- added C4: 10uf, Capacitor_SMD:C_0805_2012Metric, symbol Device:C
- added C5: 1uf, Capacitor_SMD:C_0805_2012Metric, symbol Device:C
- added C6, C7: 22pf, Capacitor_SMD:C_0805_2012Metric, symbol Device:C
- added J1: USB_B_Mini, symbol Connector:USB_B_Mini
- added R1, R2: 10k, Resistor_SMD:R_0805_2012Metric, symbol Device:R
- added R3, R4: 22, Resistor_SMD:R_0805_2012Metric, symbol Device:R
- added SW1: SW_Push, Button_Switch_SMD:SW_SPST_SKQG_WithStem, symbol Switch:SW_Push
- added Y2: Crystal_GND24, Crystal:Crystal_SMD_3225-4Pin_3.2x2.5mm, symbol Device:Crystal_GND24
Connections:
- net at U2.13 (~{RESET}): now also R2.2, SW1.2
- net +5V: now reaches U2.14 (VCC), U2.34 (VCC)
- net +5V: now also U2.2 (UVCC), U2.24 (AVCC), U2.44 (AVCC), U2.7 (VBUS), C1.1, C2.1, C3.1, C4.1, J1.1 (VBUS), R2.1
- net GND: now reaches U2.15 (GND), U2.23 (GND), U2.35 (GND), U2.43 (GND)
- net GND: now also U2.5 (UGND), C1.2, C2.2, C3.2, C4.2, C5.2, C6.2, C7.2, J1.5 (GND), R1.2, SW1.1, Y2.2, Y2.4
- net at U2.16 (XTAL2): now also C7.1, Y2.3
- net at U2.17 (XTAL1): now also C6.1, Y2.1
- net at U2.3 (D-): now also R4.1
- net at U2.33 (~{HWB}/PE2): now also R1.1
- net at U2.4 (D+): now also R3.1
- net at U2.6 (UCAP): now also C5.1
- new net D+: R3.2
- new net D-: R4.2
- no-connect marks 19 -> 12
Other:
- note added: "22 ohms from data sheet"
- note added: "AVCC is used for A/D converter, datasheet says to tie it to vcc"
- note added: "Crystal"
- note added: "Decoupling"
- note added: "Flashes a new layout when reset button is pressed"
- note added: "From data sheet"
- note added: "Keyboard matrix to be determined based on placement"
- note added: "Need to check exact decoupling cap values"
- note added: "Reset switch with pull up resistor"
- note added: "Usb will power the 5v so vbus can go to 5v"
- moved on the sheet: U2
