File: 65/65.kicad_sch (KiCad schematic)
At the start: 152 parts, among them J2 USB_C_Receptacle_USB2.0_14P, K1 KEYSW, K10 KEYSW, K11 KEYSW, K12 KEYSW, K13 KEYSW, K14 KEYSW, K15 KEYSW, K16 KEYSW, K17 KEYSW, K18 KEYSW, K19 KEYSW, K2 KEYSW, K20 KEYSW, K21 KEYSW, K22 KEYSW, K23 KEYSW, K24 KEYSW, K25 KEYSW, K26 KEYSW, K27 KEYSW, K28 KEYSW, K29 KEYSW, K3 KEYSW, K30 KEYSW, K31 KEYSW, K32 KEYSW, K33 KEYSW, K34 KEYSW, K35 KEYSW, K36 KEYSW, K37 KEYSW, K38 KEYSW, K39 KEYSW, K4 KEYSW, K40 KEYSW, K41 KEYSW, K42 KEYSW, K43 KEYSW, K44 KEYSW, K45 KEYSW, K46 KEYSW, K47 KEYSW, K48 KEYSW, K49 KEYSW, K5 KEYSW, K50 KEYSW, K51 KEYSW, K52 KEYSW, K53 KEYSW, K54 KEYSW, K55 KEYSW, K56 KEYSW, K57 KEYSW, K58 KEYSW, K59 KEYSW, K6 KEYSW, K60 KEYSW, K61 KEYSW, K62 KEYSW, K63 KEYSW, K64 KEYSW, K65 KEYSW, K66 KEYSW, K7 KEYSW, K8 KEYSW, K9 KEYSW, SW1 SW_Push, U1 USBLC6-2SC6, U2 ATmega32U4-A, Y2 Crystal_GND24

Commit message: swapped the footprint pads for the key swithces
Parts:
- J2: footprint Connector_USB:USB_C_Receptacle_HRO_TYPE-C-31-M-12 -> Connector_USB:USB_C_Receptacle_GCT_USB4105-xx-A_16P_TopMnt_Horizontal
- K1, K10, K11, K12, K13, K15, K17, K18, K19, K2, K20, K21, K22, K23, K24, K25, K26, K27, K28, K3, K30, K32, K33, K34, K35, K36, K37, K38, K39, K4, K40, K41, K42, K45, K46, K47, K48, K49, K5, K50, K51, K52, K53, K54, K56, K58, K6, K64, K65, K66, K7, K8, K9: footprint Button_Switch_Keyboard:SW_Cherry_MX_1.00u_PCB -> Footprinty:SW_Cherry_MX_1.00u_PCB
- K14: footprint Button_Switch_Keyboard:SW_Cherry_MX_2.00u_PCB -> Footprinty:SW_Cherry_MX_2.00u_PCB
- K16, K29: footprint Button_Switch_Keyboard:SW_Cherry_MX_1.50u_PCB -> Footprinty:SW_Cherry_MX_1.50u_PCB
- K31: footprint Button_Switch_Keyboard:SW_Cherry_MX_1.75u_PCB -> Footprinty:SW_Cherry_MX_1.75u_PCB
- K43, K44, K55: footprint Button_Switch_Keyboard:SW_Cherry_MX_2.25u_PCB -> Footprinty:SW_Cherry_MX_2.25u_PCB
- K57, K59, K61, K62, K63: footprint Button_Switch_Keyboard:SW_Cherry_MX_1.25u_PCB -> Footprinty:SW_Cherry_MX_1.25u_PCB
- K60: footprint Button_Switch_Keyboard:SW_Cherry_MX_6.25u_PCB -> Footprinty:SW_Cherry_MX_6.25u_PCB

Commit message: Traced monstly everything will need to fix parts
Connections:
- net Col 0: now also U2.19 (PD1); no longer U2.36 (PF7)
- net Col 1: now also U2.20 (PD2); no longer U2.32 (PC7)
- net Col 10: now also U2.31 (PC6); no longer U2.21 (PD3)
- net Col 11: now also U2.32 (PC7); no longer U2.20 (PD2)
- net Col 12: now also U2.36 (PF7); no longer U2.19 (PD1)
- net Col 2: now also U2.21 (PD3); no longer U2.31 (PC6)
- net Col 3: now also U2.22 (PD5); no longer U2.30 (PB6)
- net Col 4: now also U2.25 (PD4); no longer U2.29 (PB5)
- net Col 5: now also U2.26 (PD6); no longer U2.28 (PB4)
- net Col 7: now also U2.28 (PB4); no longer U2.26 (PD6)
- net Col 8: now also U2.29 (PB5); no longer U2.25 (PD4)
- net Col 9: now also U2.30 (PB6); no longer U2.22 (PD5)
- net D3+: no longer R4.1, U2.3 (D-)
- net GND: no longer J2.S1 (SHIELD)
- new net D3-: R4.1, U2.3 (D-)
- new net Earth: J2.S1 (SHIELD)
Changed lines of the file:
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@@
 	)
 	(junction
-		(at 111.76 279.4)
-		(diameter 0)
-		(color 0 0 0 0)
-	)
-	(junction
 		(at 318.77 356.87)
 		(diameter 0)
@@
 	(wire
 		(pts
-			(xy 111.76 279.4) (xy 107.95 279.4)
-		)
-		(stroke
-			(width 0)
-			(type default)
-		)
-	)
-	(wire
-		(pts
 			(xy 397.51 323.85) (xy 397.51 344.17)
 		)
@@
 	(wire
 		(pts
-			(xy 107.95 279.4) (xy 107.95 278.13)
-		)
-		(stroke
-			(width 0)
-			(type default)
-		)
-	)
-	(wire
-		(pts
 			(xy 347.98 364.49) (xy 347.98 367.03)
 		)
@@
 	(wire
 		(pts
-			(xy 111.76 279.4) (xy 115.57 279.4)
-		)
-		(stroke
-			(width 0)
-			(type default)
-		)
-	)
-	(wire
-		(pts
 			(xy 26.67 316.23) (xy 55.88 316.23)
 		)
@@
 	)
 	(label "Col 1"
-		(at 248.92 218.44 0)
+		(at 248.92 228.6 0)
 		(fields_autoplaced yes)
 		(effects
@@
 		)
 	)
-	(label "D3+"
+	(label "D3-"
 		(at 213.36 220.98 0)
 		(fields_autoplaced yes)
@@
 	)
 	(label "Col 2"
-		(at 248.92 215.9 0)
+		(at 248.92 231.14 0)
 		(fields_autoplaced yes)
 		(effects
@@
 	)
 	(label "Col 8"
-		(at 248.92 233.68 0)
+		(at 248.92 205.74 0)
 		(fields_autoplaced yes)
 		(effects
@@
 	)
 	(label "Col 5"
-		(at 248.92 203.2 0)
+		(at 248.92 238.76 0)
 		(fields_autoplaced yes)
 		(effects
@@
 	)
 	(label "Col 7"
-		(at 248.92 238.76 0)
+		(at 248.92 203.2 0)
 		(fields_autoplaced yes)
 		(effects
@@
 	)
 	(label "Col 0"
-		(at 248.92 266.7 0)
+		(at 248.92 226.06 0)
 		(fields_autoplaced yes)
 		(effects
@@
 	)
 	(label "Col 11"
-		(at 248.92 228.6 0)
+		(at 248.92 218.44 0)
 		(fields_autoplaced yes)
 		(effects
@@
 	)
 	(label "Col 9"
-		(at 248.92 236.22 0)
+		(at 248.92 208.28 0)
 		(fields_autoplaced yes)
 		(effects
@@
 	)
 	(label "Col 12"
-		(at 248.92 226.06 0)
+		(at 248.92 266.7 0)
 		(fields_autoplaced yes)
 		(effects
@@
 	)
 	(label "Col 10"
-		(at 248.92 231.14 0)
+		(at 248.92 215.9 0)
 		(fields_autoplaced yes)
 		(effects
@@
 	)
 	(label "Col 3"
-		(at 248.92 208.28 0)
+		(at 248.92 236.22 0)
 		(fields_autoplaced yes)
 		(effects
@@
 	)
 	(label "Col 4"
-		(at 248.92 205.74 0)
+		(at 248.92 233.68 0)
 		(fields_autoplaced yes)
 		(effects
@@
 	)
 	(symbol
+		(lib_id "power:Earth")
+		(at 107.95 278.13 0)
+		(unit 1)
+		(exclude_from_sim no)
+		(in_bom yes)
+		(on_board yes)
+		(dnp no)
+		(fields_autoplaced yes)
+		(property "Reference" "#PWR017"
+			(at 107.95 284.48 0)
+			(effects
+				(font
+					(size 1.27 1.27)
+				)
+				(hide yes)
+			)
+		)
+		(property "Value" "Earth"
+			(at 107.95 283.21 0)
+			(effects
+				(font
+					(size 1.27 1.27)
+				)
+			)
+		)
+		(property "Footprint" ""
+			(at 107.95 278.13 0)
+			(effects
+				(font
+					(size 1.27 1.27)
+				)
+				(hide yes)
+			)
+		)
+		(property "Datasheet" "~"
+			(at 107.95 278.13 0)
+			(effects
+				(font
+					(size 1.27 1.27)
+				)
+				(hide yes)
+			)
+		)
+		(property "Description" "Power symbol creates a global label with name \"Earth\""
+			(at 107.95 278.13 0)
+			(effects
+				(font
+					(size 1.27 1.27)
+				)
+				(hide yes)
+			)
+		)
+		(pin "1"
+		)
+		(instances
+			(project "65"
+				(path "/3d68b4a9-69ca-4332-b184-f6a85cbe42a9"
+					(reference "#PWR017")
+					(unit 1)
+				)
+			)
+		)
+	)
+	(symbol
 		(lib_id "power:GND")
 		(at 38.1 185.42 0)
@@
 	(symbol
 		(lib_id "power:GND")
-		(at 111.76 279.4 0)
+		(at 115.57 279.4 0)
 		(unit 1)
 		(exclude_from_sim no)
@@
 		(fields_autoplaced yes)
 		(property "Reference" "#PWR011"
-			(at 111.76 285.75 0)
+			(at 115.57 285.75 0)
 			(effects
 				(font
@@
 		)
 		(property "Value" "GND"
-			(at 111.76 284.48 0)
+			(at 115.57 284.48 0)
 			(effects
 				(font
@@
 		)
 		(property "Footprint" ""
-			(at 111.76 279.4 0)
+			(at 115.57 279.4 0)
 			(effects
 				(font
@@
 		)
 		(property "Datasheet" ""
-			(at 111.76 279.4 0)
+			(at 115.57 279.4 0)
 			(effects
 				(font
@@
 		)
 		(property "Description" "Power symbol creates a global label with name \"GND\" , ground"
-			(at 111.76 279.4 0)
+			(at 115.57 279.4 0)
 			(effects
 				(font

Commit message: Added actual keyboard values to the pcb
;)
Parts:
- K1: value KEYSW -> ESC
- K10: value KEYSW -> 9(
- K11: value KEYSW -> 0)
- K12: value KEYSW -> -_
- K13: value KEYSW -> +=
- K14: value KEYSW -> Backspace
- K15: value KEYSW -> Delete
- K16: value KEYSW -> Tab
- K17: value KEYSW -> Q
- K18: value KEYSW -> W
- K19: value KEYSW -> E
- K2: value KEYSW -> 1!
- K20: value KEYSW -> R
- K21: value KEYSW -> T
- K22: value KEYSW -> Y
- K23: value KEYSW -> U
- K24: value KEYSW -> I
- K25: value KEYSW -> O
- K26: value KEYSW -> P
- K27: value KEYSW -> [{
- K28: value KEYSW -> ]}
- K29: value KEYSW -> \|
- K3: value KEYSW -> 2@
- K30: value KEYSW -> Home
- K31: value KEYSW -> Caps
- K32: value KEYSW -> A
- K33: value KEYSW -> S
- K34: value KEYSW -> D
- K35: value KEYSW -> F
- K36: value KEYSW -> G
- K37: value KEYSW -> H
- K38: value KEYSW -> J
- K39: value KEYSW -> K
- K4: value KEYSW -> 3#
- K40: value KEYSW -> L
- K41: value KEYSW -> ;:
- K42: value KEYSW -> '"
- K43: value KEYSW -> Enter
- K44: value KEYSW -> LShift
- K45: value KEYSW -> Z
- K46: value KEYSW -> X
- K47: value KEYSW -> C
- K48: value KEYSW -> V
- K49: value KEYSW -> B
- K5: value KEYSW -> 4$
- K50: value KEYSW -> N
- K51: value KEYSW -> M
- K52: value KEYSW -> ,<
- K53: value KEYSW -> .>
- K54: value KEYSW -> /?
- K55: value KEYSW -> RShift
- K56: value KEYSW -> Up
- K57: value KEYSW -> LCtrl
- K58: value KEYSW -> Windows
- K59: value KEYSW -> LAlt
- K6: value KEYSW -> 5%
- K60: value KEYSW -> Space
- K61: value KEYSW -> RAlt
- K62: value KEYSW -> Fn
- K63: value KEYSW -> RCtrl
- K64: value KEYSW -> Left
- K65: value KEYSW -> Down
- K66: value KEYSW -> Right
- K7: value KEYSW -> 6^
- K8: value KEYSW -> 7&
- K9: value KEYSW -> 8*

Commit message: No errors on design checker, will now be moving around the traces to make the board look a lil nicer
Parts:
- J2: footprint Connector_USB:USB_C_Receptacle_GCT_USB4105-xx-A_16P_TopMnt_Horizontal -> Connector_USB:USB_C_Receptacle_HRO_TYPE-C-31-M-12
Changed lines of the file:
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@@
 			)
 		)
-		(property "Footprint" "Connector_USB:USB_C_Receptacle_GCT_USB4105-xx-A_16P_TopMnt_Horizontal"
+		(property "Footprint" "Connector_USB:USB_C_Receptacle_HRO_TYPE-C-31-M-12"
 			(at 119.38 255.27 0)
 			(effects
