File: 65/65.kicad_pcb (KiCad board)
At the start: 2 copper layers, 318.3 x 99.2 mm, 133 parts, among them K1 KEYSW, K10 KEYSW, K11 KEYSW, K12 KEYSW, K13 KEYSW, K14 KEYSW, K15 KEYSW, K16 KEYSW, K17 KEYSW, K18 KEYSW, K19 KEYSW, K2 KEYSW, K20 KEYSW, K21 KEYSW, K22 KEYSW, K23 KEYSW, K24 KEYSW, K25 KEYSW, K26 KEYSW, K27 KEYSW, K28 KEYSW, K29 KEYSW, K3 KEYSW, K30 KEYSW, K31 KEYSW, K32 KEYSW, K33 KEYSW, K34 KEYSW, K35 KEYSW, K36 KEYSW, K37 KEYSW, K38 KEYSW, K39 KEYSW, K4 KEYSW, K40 KEYSW, K41 KEYSW, K42 KEYSW, K43 KEYSW, K44 KEYSW, K45 KEYSW, K46 KEYSW, K47 KEYSW, K48 KEYSW, K49 KEYSW, K5 KEYSW, K50 KEYSW, K51 KEYSW, K52 KEYSW, K53 KEYSW, K54 KEYSW, K55 KEYSW, K56 KEYSW, K57 KEYSW, K58 KEYSW, K59 KEYSW, K6 KEYSW, K60 KEYSW, K61 KEYSW, K62 KEYSW, K63 KEYSW, K64 KEYSW, K65 KEYSW, K66 KEYSW, K7 KEYSW, K8 KEYSW, K9 KEYSW, U2 ATmega32U4-A

Commit message: almost finished the 2x2, will be working on the 65 now
Parts:
- added C1: 0.1uf, Capacitor_SMD:C_0805_2012Metric, B.Cu at (377.4, 121.9)
- added C2: 0.1uf, Capacitor_SMD:C_0805_2012Metric, B.Cu at (392.9, 127.5)
- added C3: 0.1uf, Capacitor_SMD:C_0805_2012Metric, B.Cu at (392.8, 132.5)
- added C4: 10uf, Capacitor_SMD:C_0805_2012Metric, B.Cu at (375.5, 146.2)
- added C5: 1uf, Capacitor_SMD:C_0805_2012Metric, B.Cu at (355.1, 136.6)
- added C6: 22pf, Capacitor_SMD:C_0805_2012Metric, B.Cu at (380.6, 149.8)
- added C7: 22pf, Capacitor_SMD:C_0805_2012Metric, B.Cu at (376.1, 152.7)
- added R1: 10k, Resistor_SMD:R_0805_2012Metric, B.Cu at (371.4, 127.0)
- added R2: 10k, Resistor_SMD:R_0805_2012Metric, B.Cu at (382.2, 132.3)
- added R3: 22, Resistor_SMD:R_0805_2012Metric, B.Cu at (376.4, 132.9)
- added R4: 22, Resistor_SMD:R_0805_2012Metric, B.Cu at (370.0, 137.3)
- added SW1: SW_Push, Button_Switch_SMD:SW_SPST_SKQG_WithStem, B.Cu at (361.9, 139.1)
- added Y2: Crystal_GND24, Crystal:Crystal_SMD_3225-4Pin_3.2x2.5mm, B.Cu at (357.3, 151.9)
- moved D16 63.5 mm to (61.7, 128.0)
- moved D19 62.3 mm to (123.0, 128.2)
- moved U2 3.79 mm to (347.6, 143.8), turned to -135 degrees
Connections:
- U2 pad 13: unconnected-(U2-~{RESET}-Pad13) -> Net-(U2-~{RESET})
- U2 pad 14: unconnected-(U2-VCC-Pad14) -> +5V
- U2 pad 15: unconnected-(U2-GND-Pad15)_2 -> GND
- U2 pad 16: unconnected-(U2-XTAL2-Pad16) -> Net-(U2-XTAL2)
- U2 pad 17: unconnected-(U2-XTAL1-Pad17) -> Net-(U2-XTAL1)
- U2 pad 2: unconnected-(U2-UVCC-Pad2) -> +5V
- U2 pad 23: unconnected-(U2-GND-Pad15) -> GND
- U2 pad 24: unconnected-(U2-AVCC-Pad24)_0 -> +5V
- U2 pad 3: unconnected-(U2-D--Pad3) -> Net-(U2-D-)
- U2 pad 33: unconnected-(U2-~{HWB}/PE2-Pad33) -> Net-(U2-~{HWB}/PE2)
- U2 pad 34: unconnected-(U2-VCC-Pad14)_0 -> +5V
- U2 pad 35: unconnected-(U2-GND-Pad15)_1 -> GND
- U2 pad 4: unconnected-(U2-D+-Pad4) -> Net-(U2-D+)
- U2 pad 43: unconnected-(U2-GND-Pad15)_0 -> GND
- U2 pad 44: unconnected-(U2-AVCC-Pad24) -> +5V
- U2 pad 5: unconnected-(U2-UGND-Pad5) -> GND
- U2 pad 6: unconnected-(U2-UCAP-Pad6) -> Net-(U2-UCAP)
- U2 pad 7: unconnected-(U2-VBUS-Pad7) -> +5V
Routing:
- added copper zone on B.Cu, net GND
- added copper zone on F.Cu, net GND

Commit message: Mainly did some usb stuff
Parts:
- added C8: 0.1uf, Capacitor_SMD:C_0805_2012Metric, B.Cu at (355.2, 136.6)
- added F1: Polyfuse_Small, Fuse:Fuse_1206_3216Metric, F.Cu at (188.5, 90.5)
- added J2: USB_C_Receptacle_USB2.0_14P, Connector_USB:USB_C_Receptacle_GCT_USB4105-xx-A_16P_TopMnt_Horizontal, B.Cu at (202.5, 92.2)
- added R5: 5K1, Resistor_SMD:R_0805_2012Metric, B.Cu at (206.0, 101.5)
- added R6: 5K1, Resistor_SMD:R_0805_2012Metric, B.Cu at (198.5, 101.5)
- added U1: USBLC6-2SC6, Package_TO_SOT_SMD:SOT-23-6, B.Cu at (202.5, 108.4)
- K16: footprint Button_Switch_Keyboard:SW_Cherry_MX_1.50u_Plate -> Button_Switch_Keyboard:SW_Cherry_MX_1.50u_PCB
- moved C2 61.3 mm to (335.3, 148.3)
- moved C3 44.9 mm to (351.7, 150.7), turned to 0 degrees
- moved C1 44.4 mm to (336.1, 138.3)
- moved R1 40.6 mm to (338.3, 150.6)
- moved C4 38.3 mm to (338.8, 135.1)
- moved R3 33.7 mm to (343.1, 128.1), turned to 90 degrees
- moved R4 30.3 mm to (341.1, 128.1), turned to 90 degrees
- moved R2 27.5 mm to (354.8, 134.1), turned to 0 degrees
- moved C6 25.7 mm to (357.2, 139.1), turned to 45 degrees
- moved C7 19.7 mm to (357.5, 146.3), turned to -45 degrees
- moved C5 9.45 mm to (346.4, 132.9), turned to 90 degrees
- moved Y2 9.14 mm to (358.2, 142.8), turned to -45 degrees
- moved SW1 7.02 mm to (361.4, 132.1), turned to 180 degrees
- moved U2 2.28 mm to (345.5, 142.9), turned to -90 degrees
Connections:
- net Net-(U2-UCAP) renamed /Ucap
- net Net-(U2-~{HWB}/PE2) renamed /HWB
- net Net-(U2-~{RESET}) renamed /Reset
- C6 pad 1: Net-(U2-XTAL1) -> /Xtal2
- C7 pad 1: Net-(U2-XTAL2) -> /Xtal1
- K60 pad 1: /Col 3 -> /Col 5
- K61 pad 1: /Col 4 -> /Col 8
- K62 pad 1: /Col 5 -> /Col 9
- K63 pad 1: /Col 6 -> /Col 10
- K64 pad 1: /Col 7 -> /Col 11
- K65 pad 1: /Col 8 -> /Col 12
- K66 pad 1: /Col 9 -> /Col 14
- R3 pad 1: Net-(U2-D+) -> /D3+
- R3 pad 2: /D+ -> /D2+
- R4 pad 1: Net-(U2-D-) -> /D3+
- R4 pad 2: /D- -> /D2-
- U2 pad 10: /Row 2 -> /Col 13
- U2 pad 11: /Row 3 -> /Col 14
- U2 pad 16: Net-(U2-XTAL2) -> /Xtal2
- U2 pad 17: Net-(U2-XTAL1) -> /Xtal1
- U2 pad 18: /Col 2 -> unconnected-(U2-PD0-Pad18)
- U2 pad 19: /Col 3 -> /Col 12
- U2 pad 20: /Col 4 -> /Col 11
- U2 pad 21: /Col 5 -> /Col 10
- U2 pad 22: /Col 7 -> /Col 9
- U2 pad 25: /Col 6 -> /Col 8
- U2 pad 26: /Col 8 -> /Col 7
- U2 pad 27: /Col 9 -> /Col 6
- U2 pad 28: /Row 4 -> /Col 5
- U2 pad 29: unconnected-(U2-PB5-Pad29) -> /Col 4
- U2 pad 3: Net-(U2-D-) -> /D3+
- U2 pad 30: unconnected-(U2-PB6-Pad30) -> /Col 3
- U2 pad 31: /Col 0 -> /Col 2
- U2 pad 36: unconnected-(U2-PF7-Pad36) -> /Col 0
- U2 pad 37: /Col 14 -> /Row 4
- U2 pad 38: /Col 13 -> /Row 3
- U2 pad 39: /Col 12 -> /Row 2
- U2 pad 4: Net-(U2-D+) -> /D3+
- U2 pad 40: /Col 11 -> /Row 1
- U2 pad 41: /Col 10 -> /Row 0
- U2 pad 8: /Row 0 -> unconnected-(U2-PB0-Pad8)
- U2 pad 9: /Row 1 -> unconnected-(U2-PB1-Pad9)
- Y2 pad 1: Net-(U2-XTAL1) -> /Xtal2
- Y2 pad 3: Net-(U2-XTAL2) -> /Xtal1
Routing:
- net /D2+: track 0.00 -> 154.0 mm
- net /D2-: track 0.00 -> 153.9 mm
- net /Col 1: track 0.00 -> 101.2 mm
- net /Col 0: track 0.00 -> 90.4 mm
- net /Col 12: track 0.00 -> 88.5 mm
- net /Col 5: track 0.00 -> 87.0 mm
- net /Col 11: track 0.00 -> 86.0 mm
- net /Col 9: track 0.00 -> 83.7 mm
- net /Col 10: track 0.00 -> 82.9 mm
- net /Col 8: track 0.00 -> 77.5 mm
- net /Col 7: track 0.00 -> 71.0 mm
- net /Col 2: track 0.00 -> 67.2 mm
- net /Col 6: track 0.00 -> 67.0 mm
- net /Col 4: track 0.00 -> 67.0 mm
- net /Col 3: track 0.00 -> 67.0 mm
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
Commit message: swapped the footprint pads for the key swithces
Parts:
- removed D49, D60: D, Diode_SMD:D_SOD-123
- removed K46: KEYSW, Button_Switch_Keyboard:SW_Cherry_MX_1.00u_PCB
- removed K59, K62: KEYSW, Button_Switch_Keyboard:SW_Cherry_MX_1.25u_PCB
- F1: moved to B.Cu
- K1, K10, K11, K12, K13, K15, K17, K18, K19, K2, K20, K21, K22, K23, K24, K25, K26, K27, K28, K3, K30, K32, K33, K34, K35, K36, K37, K38, K39, K4, K40, K41, K42, K45, K47, K48, K49, K5, K50, K51, K52, K53, K54, K56, K58, K6, K64, K65, K66, K7, K8, K9: footprint Button_Switch_Keyboard:SW_Cherry_MX_1.00u_PCB -> Footprinty:SW_Cherry_MX_1.00u_PCB
- K14: footprint Button_Switch_Keyboard:SW_Cherry_MX_2.00u_PCB -> Footprinty:SW_Cherry_MX_2.00u_PCB
- K16, K29: footprint Button_Switch_Keyboard:SW_Cherry_MX_1.50u_PCB -> Footprinty:SW_Cherry_MX_1.50u_PCB
- K31: footprint Button_Switch_Keyboard:SW_Cherry_MX_1.75u_PCB -> Footprinty:SW_Cherry_MX_1.75u_PCB
- K43, K44, K55: footprint Button_Switch_Keyboard:SW_Cherry_MX_2.25u_PCB -> Footprinty:SW_Cherry_MX_2.25u_PCB
- K57, K61, K63: footprint Button_Switch_Keyboard:SW_Cherry_MX_1.25u_PCB -> Footprinty:SW_Cherry_MX_1.25u_PCB
- K60: footprint Button_Switch_Keyboard:SW_Cherry_MX_6.25u_PCB -> Footprinty:SW_Cherry_MX_6.25u_PCB
- moved F1 33.4 mm to (221.5, 95.9)
- moved SW1 26.8 mm to (359.0, 158.8), turned to 0 degrees
- moved R5 0.51 mm to (205.5, 101.4)
- moved R6 0.51 mm to (199.0, 101.4)
Routing:
- net /Col 1: track 101.2 -> 0.00 mm
- net /Col 12: track 88.5 -> 0.00 mm
- net /Col 5: track 87.0 -> 0.00 mm
- net /Col 11: track 86.0 -> 0.00 mm
- net /Col 0: track 90.4 -> 5.33 mm
- net /Col 9: track 83.7 -> 0.00 mm
- net /Col 10: track 82.9 -> 0.00 mm
- net /Col 8: track 77.5 -> 0.00 mm
- net /Col 7: track 71.0 -> 0.00 mm
- net /Col 2: track 67.2 -> 0.00 mm
- net /Col 6: track 67.0 -> 0.00 mm
- net /Col 4: track 67.0 -> 0.00 mm
- net /Col 3: track 67.0 -> 0.00 mm
- net +5V: track 16.6 -> 35.3 mm
- net /Col 13: track 14.3 -> 0.00 mm
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
Commit message: Initial traces of switches
Parts:
- added D49: D, Diode_SMD:D_SOD-123, B.Cu at (181.8, 166.1)
- added D60: D, Diode_SMD:D_SOD-123, B.Cu at (179.4, 184.9)
- added K46: KEYSW, Footprinty:SW_Cherry_MX_1.00u_PCB, F.Cu at (124.0, 156.4)
- added K59: KEYSW, Footprinty:SW_Cherry_MX_1.25u_PCB, F.Cu at (107.3, 175.5)
- added K62: KEYSW, Footprinty:SW_Cherry_MX_1.25u_PCB, F.Cu at (274.0, 175.5)
- moved D13 9.11 mm to (291.3, 109.0)
- moved D9 8.81 mm to (215.1, 109.0)
- moved D46 8.62 mm to (124.6, 166.1)
- moved D10 8.36 mm to (234.2, 109.0)
- moved D11 8.31 mm to (253.2, 109.0)
- moved D7 8.21 mm to (177.0, 109.0)
- moved D63 7.85 mm to (298.4, 185.2)
- moved D5 7.71 mm to (138.9, 109.0)
- moved D12 7.56 mm to (272.3, 109.0)
- moved D52 7.42 mm to (238.9, 166.1)
- moved D40 7.34 mm to (248.4, 147.1)
- moved D42 7.24 mm to (286.5, 147.1)
- moved D65 7.23 mm to (338.9, 185.2)
- moved D41 7.09 mm to (267.5, 147.1)
- moved D6 7.06 mm to (158.0, 109.0)
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Routing:
- net /Row 4: track 5.25 -> 301.1 mm
- net /Row 1: track 5.62 -> 262.1 mm
- net /Row 2: track 5.29 -> 253.9 mm
- net /Row 0: track 5.62 -> 244.7 mm
- net /Row 3: track 5.12 -> 240.3 mm
- net +5V: track 35.3 -> 199.1 mm
- net /Col 12: track 0.00 -> 110.8 mm
- net /Col 11: track 0.00 -> 102.8 mm
- net /Col 10: track 0.00 -> 102.8 mm
- net /Col 1: track 0.00 -> 102.3 mm
- net /Col 2: track 0.00 -> 99.1 mm
- net /Col 9: track 0.00 -> 97.5 mm
- net /Col 8: track 0.00 -> 93.3 mm
- net /Col 5: track 0.00 -> 87.5 mm
- net /Col 0: track 5.33 -> 90.4 mm
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
Commit message: Traced monstly everything will need to fix parts
Parts:
- moved D64 12.6 mm to (325.1, 173.8), turned to -90 degrees
- moved D66 12.5 mm to (363.1, 173.8), turned to -90 degrees
- moved D58 12.5 mm to (91.6, 173.8), turned to -90 degrees
- moved D61 12.5 mm to (255.9, 173.8), turned to -90 degrees
- moved D63 12.5 mm to (303.5, 173.8), turned to -90 degrees
- moved D59 12.5 mm to (113.0, 173.8), turned to -90 degrees
- moved D62 12.5 mm to (279.6, 173.8), turned to -90 degrees
- moved D57 12.4 mm to (70.3, 173.9), turned to -90 degrees
- moved D60 12.2 mm to (184.3, 173.8), turned to -90 degrees
- moved D65 11.8 mm to (341.9, 173.8), turned to -90 degrees
- moved SW1 3.40 mm to (359.8, 162.1)
- moved C1 1.28 mm to (335.1, 137.5)
- moved D29 0.85 mm to (324.7, 128.0)
Connections:
- J2 pad S1: GND -> Earth
- R4 pad 1: /D3+ -> /D3-
- U2 pad 19: /Col 12 -> /Col 0
- U2 pad 20: /Col 11 -> /Col 1
- U2 pad 21: /Col 10 -> /Col 2
- U2 pad 22: /Col 9 -> /Col 3
- U2 pad 25: /Col 8 -> /Col 4
- U2 pad 26: /Col 7 -> /Col 5
- U2 pad 28: /Col 5 -> /Col 7
- U2 pad 29: /Col 4 -> /Col 8
- U2 pad 3: /D3+ -> /D3-
- U2 pad 30: /Col 3 -> /Col 9
- U2 pad 31: /Col 2 -> /Col 10
- U2 pad 32: /Col 1 -> /Col 11
- U2 pad 36: /Col 0 -> /Col 12
Routing:
- net /Col 0: track 90.4 -> 442.9 mm, vias 0 -> 1
- net /Col 1: track 102.3 -> 439.8 mm, vias 0 -> 1
- net /Col 2: track 99.1 -> 413.3 mm, vias 0 -> 1
- net /Col 3: track 67.0 -> 354.4 mm, vias 0 -> 1
- net /Col 4: track 67.0 -> 328.7 mm, vias 0 -> 1
- net /Col 5: track 87.5 -> 311.9 mm, vias 0 -> 1
- net /Col 6: track 67.0 -> 287.5 mm, vias 0 -> 1
- net /Col 7: track 67.0 -> 267.4 mm, vias 0 -> 1
- net /Col 8: track 93.3 -> 247.6 mm, vias 0 -> 1
- net /Col 9: track 97.5 -> 227.2 mm, vias 0 -> 1
- net /Col 10: track 102.8 -> 206.9 mm, vias 0 -> 1
- net +5V: track 199.1 -> 290.8 mm, vias 0 -> 2
- net /Row 0: track 244.7 -> 335.3 mm, vias 0 -> 6
- net /Col 14: track 19.0 -> 104.9 mm, vias 0 -> 1
- net /Col 11: track 102.8 -> 187.8 mm, vias 0 -> 1
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- added copper zone on B.Cu, net Earth
- added copper zone on F.Cu, net Earth
Other:
- board size 318.3 x 99.2 mm -> 318.3 x 104.1 mm

Commit message: Added actual keyboard values to the pcb
;)
Parts:
- K1: value KEYSW -> ESC
- K10: value KEYSW -> 9(
- K11: value KEYSW -> 0)
- K12: value KEYSW -> -_
- K13: value KEYSW -> +=
- K14: value KEYSW -> Backspace
- K15: value KEYSW -> Delete
- K16: value KEYSW -> Tab
- K17: value KEYSW -> Q
- K18: value KEYSW -> W
- K19: value KEYSW -> E
- K2: value KEYSW -> 1!
- K20: value KEYSW -> R
- K21: value KEYSW -> T
- K22: value KEYSW -> Y
- K23: value KEYSW -> U
- K24: value KEYSW -> I
- K25: value KEYSW -> O
- K26: value KEYSW -> P
- K27: value KEYSW -> [{
- K28: value KEYSW -> ]}
- K29: value KEYSW -> \|
- K3: value KEYSW -> 2@
- K30: value KEYSW -> Home
- K31: value KEYSW -> Caps
- K32: value KEYSW -> A
- K33: value KEYSW -> S
- K34: value KEYSW -> D
- K35: value KEYSW -> F
- K36: value KEYSW -> G
- K37: value KEYSW -> H
- K38: value KEYSW -> J
- K39: value KEYSW -> K
- K4: value KEYSW -> 3#
- K40: value KEYSW -> L
- K41: value KEYSW -> ;:
- K42: value KEYSW -> '"
- K43: value KEYSW -> Enter
- K44: value KEYSW -> LShift
- K45: value KEYSW -> Z
- K46: value KEYSW -> X
- K47: value KEYSW -> C
- K48: value KEYSW -> V
- K49: value KEYSW -> B
- K5: value KEYSW -> 4$
- K50: value KEYSW -> N
- K51: value KEYSW -> M
- K52: value KEYSW -> ,<
- K53: value KEYSW -> .>
- K54: value KEYSW -> /?
- K55: value KEYSW -> RShift
- K56: value KEYSW -> Up
- K57: value KEYSW -> LCtrl
- K58: value KEYSW -> Windows
- K59: value KEYSW -> LAlt
- K6: value KEYSW -> 5%
- K60: value KEYSW -> Space
- K61: value KEYSW -> RAlt
- K62: value KEYSW -> Fn
- K63: value KEYSW -> RCtrl
- K64: value KEYSW -> Left
- K65: value KEYSW -> Down
- K66: value KEYSW -> Right
- K7: value KEYSW -> 6^
- K8: value KEYSW -> 7&
- K9: value KEYSW -> 8*
Other:
- outline, holes or cut-outs redrawn
